Commit message: Better inertia for Kabuto rover in the gazebo simulation.

File: hotwheels_ws/src/hotwheels_description/gazebo/gazebo.urdf.xacro (robot description, xacro)
@@ -7,3 +7,10 @@
   </plugin>
 </gazebo>
+<gazebo reference="base_link">
+    <turnGravityOff>false</turnGravityOff>
+  </gazebo>
+  <gazebo reference="chassis_link">
+   <!-- <material>Gazebo/DarkGrey</material-->
+    <turnGravityOff>false</turnGravityOff>
+  </gazebo>
 </robot>

File: hotwheels_ws/src/hotwheels_description/robots/kabuto.urdf.xacro (robot description, xacro)
@@ -30,5 +30,5 @@
       <!-- Center of mass -->
       <origin xyz="0.012  0.002 0.067" rpy="0 0 0"/>
-      <mass value="16.523"/>
+      <mass value="6.523"/>
       <!-- Moments of inertia: ( chassis without wheels ) -->
       <inertia
@@ -50,7 +50,10 @@
     <inertial>
         <origin xyz="0 0 0" rpy="0 0 0"/>
-          <mass value="1"/>
-           <inertia ixx="1.0" ixy="0.0" ixz="0.0" iyy="1.0" iyz="0.0" izz="1.0"/>
-     </inertial>
+        <mass value="0.477"/>
+        <inertia
+          ixx="0.0013" ixy="0" ixz="0"
+          iyy="0.0024" iyz="0"
+          izz="0.0013"/>
+      </inertial>
     <!-- <inertial>
       <origin xyz="0 0 0" rpy="0 0 0"/>
